Commit message: fixed robotiq_gripper moveit config

File: robotiq_gripper_moveit_config/config/robotiq_85_gripper.ros2_control.xacro (robot description, xacro)
@@ -15,4 +15,39 @@
                 <state_interface name="velocity"/>
             </joint>
+            <joint name="robotiq_85_right_knuckle_joint">
+                <param name="mimic">robotiq_85_left_knuckle_joint</param>
+                <param name="multiplier">1</param>
+                <command_interface name="position" />
+                <state_interface name="position"/>
+                <state_interface name="velocity"/>
+            </joint>
+            <joint name="robotiq_85_left_inner_knuckle_joint">
+                <param name="mimic">robotiq_85_left_knuckle_joint</param>
+                <param name="multiplier">1</param>
+                <command_interface name="position" />
+                <state_interface name="position"/>
+                <state_interface name="velocity"/>
+            </joint>
+            <joint name="robotiq_85_right_inner_knuckle_joint">
+                <param name="mimic">robotiq_85_left_knuckle_joint</param>
+                <param name="multiplier">1</param>
+                <command_interface name="position" />
+                <state_interface name="position"/>
+                <state_interface name="velocity"/>
+            </joint>
+            <joint name="robotiq_85_left_finger_tip_joint">
+                <param name="mimic">robotiq_85_left_knuckle_joint</param>
+                <param name="multiplier">-1</param>
+                <command_interface name="position" />
+                <state_interface name="position"/>
+                <state_interface name="velocity"/>
+            </joint>
+            <joint name="robotiq_85_right_finger_tip_joint">
+                <param name="mimic">robotiq_85_left_knuckle_joint</param>
+                <param name="multiplier">-1</param>
+                <command_interface name="position" />
+                <state_interface name="position"/>
+                <state_interface name="velocity"/>
+            </joint>
         </ros2_control>
     </xacro:macro>
